Commit message: Updated URDF with new origins
Attempt to fix problem with urdf render

File: j2_prototype3_3/urdf/j2_prototype3_3.urdf (robot description, URDF)
Before this commit: robot j2_prototype3_3, 7 links, 6 joints
Links:
- link Link_0: mass 0.88481 -> 0.884810555483961
- link Link_2: mass 1.6567 -> 1.65666298237922
- link base_link: mass 2.04931359707062 -> 2.0493
Joints:
- joint Base_Rotate: axis 1 0 0 -> 0 0 1; origin xyz=0.0483 0.1263 0 rpy=-1.5708 0 -1.5708 -> xyz=0.0483 0 -0.1263 rpy=0 0 -1.5708
- joint Effector_Limb: origin xyz=0.0403 0.0383 0.2 rpy=0 0 -1.5708 -> xyz=0.040299998474171 0.038300000000004 0.199999999999992 rpy=0 0 -1.5707963267949
- joint Limb_1: origin xyz=0.126300000762939 0 -0.0383 rpy=0 -1.5707963267949 0 -> xyz=0 -0.0382999999999991 0.126300000762939 rpy=0 0 1.5707963267949
- joint Limb_3: origin xyz=0.041578 0.037604 0.20106 rpy=0 0 -1.5708 -> xyz=0.041577919602976 0.037603596411357 0.201058687851851 rpy=0 0 -1.5707963267949
- joint Limb_4: origin xyz=0.037604 0.039022 0.19894 rpy=0 0 -1.5708 -> xyz=0.037603596411366 0.039022070574184 0.198941312148156 rpy=0 0 -1.5707963267949
